File: LED_Matrix_Driver/LED_Matrix_Driver.sch (KiCad schematic (older format))
At the start: 65 parts, among them J1 Screw_Terminal_01x02, J2 LED Anode Rows, J3 Columns 24-31 LED Cathodes, J4 Columns 16-23 LED Cathodes, J5 Columns 8-15 LED Cathodes, J6 Columns 0-7 LED Cathodes, U1 ESP32-DEVKITC-32E, U2 74HCT244, U3 MIC2981, U4 74HC238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

Commit message: Started work on including an ATmega328P in the schematic
Parts:
- removed C1, C2, C3, C4: 0.1uF, Capacitor_THT:C_Axial_L3.8mm_D2.6mm_P7.50mm_Horizontal, symbol Device:C_Small
- removed R1, R2, R3, R4, R5, R6, R7: 1M, Resistor_THT:R_Axial_DIN0204_L3.6mm_D1.6mm_P7.62mm_Horizontal, symbol Device:R_Small_US
- removed U2: 74HCT244, Package_DIP:DIP-20_W7.62mm_Socket, symbol 74xx:74HCT244
- added U?: ATmega328P-PU, Package_DIP:DIP-28_W7.62mm, symbol MCU_Microchip_ATmega:ATmega328P-PU
Connections:
- net +5V: now also U1.19 (5V)
- net at U5.1 (STR), U6.1 (STR), U7.1 (STR)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: now also U?.2 (PD0)
- net at U5.15 (EO), U6.15 (EO), U7.15 (EO)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: now also U?.5 (PD3)
- net at U5.2 (DATA): now also U?.3 (PD1)
- net at U5.3 (CLK), U6.3 (CLK), U7.3 (CLK)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: now also U?.4 (PD2)
- net at U4.1 (A0): now also U?.6 (PD4)
- net at U4.2 (A1): now also U?.11 (PD5)
- net at U4.3 (A2): now also U?.12 (PD6)
- new net: U?.22 (GND), U?.8 (GND)
Other:
- note removed: "Note: Purpose of 74HCT244 is to translate 3V3 \nlogic from ESP32 to 5V logic for the control ICs. \nUnidirectional operation only."
- moved on the sheet: U1, U4
