File: LED_Matrix_8x32_v2/LED_Matrix_8x32_v2.kicad_pcb (KiCad board)
At the start: 2 copper layers, 261 parts, among them J10 Screw_Terminal_01x08, J11 Screw_Terminal_01x08, J7 Screw_Terminal_01x08, J8 Screw_Terminal_01x08, J9 Screw_Terminal_01x08

Commit message: Created Gerber plots of new driver board design, button board, and new LED board As of 12/15/2023, all three PCBs have been submitted to JLCPCB for manufacturing.
Parts:
- added REF**: MountingHole_2.2mm_M2, MountingHole:MountingHole_2.2mm_M2, F.Cu at (247.7, 16.5)
- added REF**: , MountingHole:MountingHole_2.2mm_M2, F.Cu at (247.7, 76.2)
- added REF**: , MountingHole:MountingHole_2.2mm_M2, F.Cu at (15.9, 76.2)
- added REF**: MountingHole_2.2mm_M2, MountingHole:MountingHole_2.2mm_M2, F.Cu at (15.9, 16.5)
- moved D202 227.8 mm to (198.8, 33.0), turned to 90 degrees
- moved D186 226.2 mm to (184.8, 33.0), turned to 90 degrees
- moved D82 225.6 mm to (94.0, 33.0), turned to 90 degrees
- moved D179 224.3 mm to (177.8, 40.0), turned to 90 degrees
- moved D130 224.1 mm to (135.9, 33.0), turned to 90 degrees
- moved D250 219.7 mm to (240.7, 33.0), turned to 90 degrees
- moved D58 217.2 mm to (73.0, 33.0), turned to 90 degrees
- moved D227 213.4 mm to (219.7, 40.0), turned to 90 degrees
- moved D180 212.8 mm to (177.8, 47.0), turned to 90 degrees
- moved D226 210.9 mm to (219.7, 33.0), turned to 90 degrees
- moved D178 208.5 mm to (177.8, 33.0), turned to 90 degrees
- moved D157 207.5 mm to (156.8, 54.0), turned to 90 degrees
- moved D172 206.8 mm to (170.8, 47.0), turned to 90 degrees
- moved D156 205.4 mm to (156.8, 47.0), turned to 90 degrees
- moved D48 204.6 mm to (59.1, 74.9), turned to 90 degrees
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Routing:
- net Net-(D17-Pad1): track 78.0 -> 75.4 mm
- net Net-(D10-Pad1): track 76.5 -> 74.0 mm
- net Net-(D1-Pad1): track 75.1 -> 72.5 mm
- net Net-(D65-Pad1): track 94.4 -> 95.6 mm, vias 0 -> 1
- net Net-(D137-Pad1): track 123.9 -> 122.9 mm
- net Net-(D121-Pad1): track 118.8 -> 117.8 mm
- net Net-(D73-Pad1): track 97.9 -> 96.9 mm
- net Net-(D41-Pad1): track 85.8 -> 84.8 mm
- net Net-(D57-Pad1): track 92.8 -> 91.7 mm
- net Net-(D89-Pad1): track 104.9 -> 103.8 mm
- net Net-(D105-Pad1): track 111.8 -> 110.8 mm
- net Net-(D169-Pad1): track 137.9 -> 136.8 mm
- net Net-(D233-Pad1): track 163.9 -> 162.9 mm
- net Net-(D201-Pad1): track 150.0 -> 148.9 mm
- net Net-(D217-Pad1): track 156.9 -> 155.9 mm
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Other:
- board outline added: 239.4 x 67.6 mm
- board text added: "(C) Matt Bowen 2023"
- board text added: "00"
- board text added: "01"
- board text added: "02"
- board text added: "03"
- board text added: "04"
- board text added: "05"
- board text added: "06"
- board text added: "07"
- board text added: "08"
- board text added: "09"
- board text added: "10"
- board text added: "11"
- board text added: "12"
- board text added: "13"
- board text added: "14"
- board text added: "15"
- board text added: "16"
- board text added: "17"
- board text added: "18"
- board text added: "19"
- board text added: "20"
- board text added: "21"
- board text added: "22"
- board text added: "23"
- board text added: "24"
- board text added: "25"
- board text added: "26"
- board text added: "27"
- board text added: "28"
- board text added: "29"
- board text added: "30"
- board text added: "31"
- board text added: "8x32 LED Matrix V2"
- board text added: "A"
- board text added: "B"
- board text added: "C"
- board text added: "D"
- board text added: "E"
- board text added: "F"
- board text added: "G"
- board text added: "H"
