File: LED_Matrix_8x32_v2/LED_Matrix_8x32_v2.sch (KiCad schematic (older format))
At the start: 261 parts, among them J10 Screw_Terminal_01x08, J11 Screw_Terminal_01x08, J7 Screw_Terminal_01x08, J8 Screw_Terminal_01x08, J9 Screw_Terminal_01x08

Commit message: Created Gerber plots of new driver board design, button board, and new LED board As of 12/15/2023, all three PCBs have been submitted to JLCPCB for manufacturing.
Parts:
- renumbered J7 to J1, J8 to J2, J9 to J3, J10 to J4, J11 to J5
Changed lines of the file:
@@
 Connection ~ 2900 2550
 $Comp
-L Connector:Screw_Terminal_01x08 J7
+L Connector:Screw_Terminal_01x08 J1
 U 1 1 6670CCDF
 P 2050 1150
-F 0 "J7" H 1968 1667 50  0000 C CNN
+F 0 "J1" H 1968 1667 50  0000 C CNN
 F 1 "Screw_Terminal_01x08" H 1968 1576 50  0000 C CNN
 F 2 "TerminalBlock_4Ucon:TerminalBlock_4Ucon_1x08_P3.50mm_Horizontal" H 2050 1150 50  0001 C CNN
@@
 Connection ~ 3500 2800
 $Comp
-L Connector:Screw_Terminal_01x08 J8
+L Connector:Screw_Terminal_01x08 J2
 U 1 1 68EAF101
 P 2900 3200
-F 0 "J8" V 2900 3650 50  0000 R CNN
+F 0 "J2" V 2900 3650 50  0000 R CNN
 F 1 "Screw_Terminal_01x08" V 3000 3550 50  0000 R CNN
 F 2 "TerminalBlock_4Ucon:TerminalBlock_4Ucon_1x08_P3.50mm_Horizontal" H 2900 3200 50  0001 C CNN
@@
 	4500 2950 4400 2950
 $Comp
-L Connector:Screw_Terminal_01x08 J9
+L Connector:Screw_Terminal_01x08 J3
 U 1 1 6B9D543C
 P 4100 3200
-F 0 "J9" V 4100 3650 50  0000 R CNN
+F 0 "J3" V 4100 3650 50  0000 R CNN
 F 1 "Screw_Terminal_01x08" V 4200 3550 50  0000 R CNN
 F 2 "TerminalBlock_4Ucon:TerminalBlock_4Ucon_1x08_P3.50mm_Horizontal" H 4100 3200 50  0001 C CNN
@@
 	5700 2950 5600 2950
 $Comp
-L Connector:Screw_Terminal_01x08 J10
+L Connector:Screw_Terminal_01x08 J4
 U 1 1 6BAD41D2
 P 5300 3200
-F 0 "J10" V 5300 3650 50  0000 R CNN
+F 0 "J4" V 5300 3650 50  0000 R CNN
 F 1 "Screw_Terminal_01x08" V 5400 3550 50  0000 R CNN
 F 2 "TerminalBlock_4Ucon:TerminalBlock_4Ucon_1x08_P3.50mm_Horizontal" H 5300 3200 50  0001 C CNN
@@
 	6900 2950 6800 2950
 $Comp
-L Connector:Screw_Terminal_01x08 J11
+L Connector:Screw_Terminal_01x08 J5
 U 1 1 6BBE4F86
 P 6500 3200
-F 0 "J11" V 6500 3650 50  0000 R CNN
+F 0 "J5" V 6500 3650 50  0000 R CNN
 F 1 "Screw_Terminal_01x08" V 6600 3550 50  0000 R CNN
 F 2 "TerminalBlock_4Ucon:TerminalBlock_4Ucon_1x08_P3.50mm_Horizontal" H 6500 3200 50  0001 C CNN
